File: eink-breakout.kicad_sch (KiCad schematic)
At the start: 25 parts, among them J1 MCU, Q1 IRLML0100, U1 WAVESHARE_4_2_INCH_EINK_DISPL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

Commit message: DNP of R1
Datasheet showed R1 attached to gate of mosfet, this was
incorrect. Fixed in this version by not populating footprint.
Other:
- note added: "Do Not Populate"
- note added: "This resistor was shown on the datasheet example circuit. It is unneeded."
- title: (none) -> Eink-Breakout
Changed lines of the file:
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@@
 	(generator_version "9.0")
 	(paper "A4")
+	(title_block
+		(title "Eink-Breakout")
+		(rev "v1.1")
+	)
+	(rectangle
+		(start 156.21 81.28)
+		(end 177.8 106.68)
+		(stroke
+			(width 0)
+			(type solid)
+		)
+		(fill
+			(type color)
+			(color 194 194 194 1)
+		)
+	)
+	(text "Do Not Populate"
+		(exclude_from_sim no)
+		(at 166.37 83.82 0)
+		(effects
+			(font
+				(size 1.27 1.27)
+				(thickness 0.254)
+				(bold yes)
+			)
+		)
+	)
+	(text "This resistor was shown\non the datasheet example\ncircuit. It is unneeded."
+		(exclude_from_sim no)
+		(at 167.64 101.6 0)
+		(effects
+			(font
+				(size 1.016 1.016)
+				(thickness 0.1588)
+			)
+		)
+	)
 	(text "EINK DISPLAY"
 		(exclude_from_sim no)
